File: KiCad/ISA8_Ethernet.kicad_pcb (KiCad board)
At the start: 2 copper layers, 104.1 x 74.9 mm, 34 parts, among them J1 RJMG1BD3B8K1ANR, J2 MEM_EXT, SW1 CONFIG, SW2 IRQ, SW3 IO_ADDR, SW4 ROM_ADDR, U1 RTL8019AS, U2 SST39SF040, U3 93LC46C, Y1 20MHz

Commit message: Rework
Parts:
- removed J2: MEM_EXT, My_Components:Conn_Pin_Header_20x2_2.54mm
- removed REF**: OSHW-Logo_5.7x6mm_SilkScreen, Symbol:OSHW-Logo_5.7x6mm_SilkScreen
- removed REF**: KiCad-Logo2_5mm_SilkScreen, Symbol:KiCad-Logo2_5mm_SilkScreen
- removed RN1, RN2, RN3, RN4: 10k, Resistor_SMD:R_Array_Convex_4x0603
- removed SW1: CONFIG, My_Components:Switch_DIP_2_Positions
- removed SW2: IRQ, My_Components:Switch_DIP_2_Positions
- removed SW3: IO_ADDR, My_Components:Switch_DIP_4_Positions
- removed SW4: ROM_ADDR, My_Components:Switch_DIP_5_Positions
- added J10: Conn_02x05_Odd_Even, Connector_PinHeader_2.54mm:PinHeader_2x05_P2.54mm_Vertical, F.Cu at (159.7, 65.6)
- added J4: Conn_02x02_Odd_Even, Connector_PinHeader_2.54mm:PinHeader_2x02_P2.54mm_Vertical, F.Cu at (126.6, 65.6)
- added J7: Conn_02x02_Odd_Even, Connector_PinHeader_2.54mm:PinHeader_2x02_P2.54mm_Vertical, F.Cu at (133.9, 65.6)
- added J9: Conn_02x04_Odd_Even, Connector_PinHeader_2.54mm:PinHeader_2x04_P2.54mm_Vertical, F.Cu at (142.0, 65.6)
- added R10: 10K, Resistor_THT:R_Axial_DIN0207_L6.3mm_D2.5mm_P10.16mm_Horizontal, F.Cu at (141.1, 78.7)
- added R11: 10K, Resistor_THT:R_Axial_DIN0207_L6.3mm_D2.5mm_P10.16mm_Horizontal, F.Cu at (144.2, 78.7)
- added R12: 10K, Resistor_THT:R_Axial_DIN0207_L6.3mm_D2.5mm_P10.16mm_Horizontal, F.Cu at (147.3, 78.7)
- added R13: 10K, Resistor_THT:R_Axial_DIN0207_L6.3mm_D2.5mm_P10.16mm_Horizontal, F.Cu at (150.4, 78.7)
- added R14: 10K, Resistor_THT:R_Axial_DIN0207_L6.3mm_D2.5mm_P10.16mm_Horizontal, F.Cu at (158.6, 78.7)
- added R15: 10K, Resistor_THT:R_Axial_DIN0207_L6.3mm_D2.5mm_P10.16mm_Horizontal, F.Cu at (161.7, 78.7)
- added R16: 10K, Resistor_THT:R_Axial_DIN0207_L6.3mm_D2.5mm_P10.16mm_Horizontal, F.Cu at (164.8, 78.7)
- added R17: 10K, Resistor_THT:R_Axial_DIN0207_L6.3mm_D2.5mm_P10.16mm_Horizontal, F.Cu at (167.9, 78.7)
- added R18: 10K, Resistor_THT:R_Axial_DIN0207_L6.3mm_D2.5mm_P10.16mm_Horizontal, F.Cu at (154.4, 89.7)
- added R19: 10K, Resistor_THT:R_Axial_DIN0207_L6.3mm_D2.5mm_P10.16mm_Horizontal, F.Cu at (171.0, 78.7)
- added R4: 10K, Resistor_THT:R_Axial_DIN0207_L6.3mm_D2.5mm_P10.16mm_Horizontal, F.Cu at (126.2, 78.8)
- added R5: 10K, Resistor_THT:R_Axial_DIN0207_L6.3mm_D2.5mm_P10.16mm_Horizontal, F.Cu at (129.4, 78.8)
- added R8: 10K, Resistor_THT:R_Axial_DIN0207_L6.3mm_D2.5mm_P10.16mm_Horizontal, F.Cu at (133.7, 78.8)
- added R9: 10K, Resistor_THT:R_Axial_DIN0207_L6.3mm_D2.5mm_P10.16mm_Horizontal, F.Cu at (136.8, 78.8)
- C1, C2, C3, C4, C5, C6, C7, C8: footprint Capacitor_SMD:C_0603_1608Metric_Pad1.08x0.95mm_HandSolder -> Capacitor_THT:C_Disc_D7.0mm_W2.5mm_P5.00mm
- C10, C9: footprint Capacitor_Tantalum_SMD:CP_EIA-3528-15_AVX-H_Pad1.50x2.35mm_HandSolder -> Capacitor_THT:CP_Radial_D6.3mm_P2.50mm
- R1, R2, R3, R6, R7: footprint Resistor_SMD:R_0603_1608Metric_Pad0.98x0.95mm_HandSolder -> Resistor_THT:R_Axial_DIN0207_L6.3mm_D2.5mm_P10.16mm_Horizontal
- moved C1 27.4 mm to (193.3, 72.1)
- moved C2 25.0 mm to (193.4, 68.5)
- moved R2 23.9 mm to (200.5, 106.0)
- moved C4 17.3 mm to (182.6, 97.8), turned to -90 degrees
- moved R7 16.4 mm to (184.9, 75.4), turned to 90 degrees
- moved Y1 15.9 mm to (180.2, 70.6)
- moved C9 14.0 mm to (179.0, 121.1), turned to 0 degrees
- moved C8 12.9 mm to (124.6, 90.6)
- moved R6 12.6 mm to (125.0, 106.1)
- moved U3 10.5 mm to (127.1, 96.2)
- moved C5 10.2 mm to (160.0, 89.3), turned to 0 degrees
- moved R1 9.68 mm to (194.6, 78.6)
- moved U2 9.07 mm to (113.1, 93.5)
- moved U1 7.67 mm to (150.4, 102.7)
- moved C7 6.57 mm to (120.8, 71.4)
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Connections:
- net /~BCS renamed /~{BCS}
- net /~IOCS16 renamed /~{IOCS16}
- net /~IOR renamed /~{IOR}
- net /~IOW renamed /~{IOW}
- net /~SMEMR renamed /~{SMEMR}
- net /~SMEMW renamed /~{SMEMW}
- BUS1 pad 15: Net-(BUS1-Pad15) -> unconnected-(BUS1-DACK3-Pad15)
- BUS1 pad 16: Net-(BUS1-Pad16) -> unconnected-(BUS1-DRQ3-Pad16)
- BUS1 pad 17: Net-(BUS1-Pad17) -> unconnected-(BUS1-DACK1-Pad17)
- BUS1 pad 18: Net-(BUS1-Pad18) -> unconnected-(BUS1-DRQ1-Pad18)
- BUS1 pad 19: Net-(BUS1-Pad19) -> unconnected-(BUS1-DACK0-Pad19)
- BUS1 pad 20: Net-(BUS1-Pad20) -> unconnected-(BUS1-CLK-Pad20)
- BUS1 pad 21: Net-(BUS1-Pad21) -> unconnected-(BUS1-IRQ7-Pad21)
- BUS1 pad 22: Net-(BUS1-Pad22) -> unconnected-(BUS1-IRQ6-Pad22)
- BUS1 pad 26: Net-(BUS1-Pad26) -> unconnected-(BUS1-DACK2-Pad26)
- BUS1 pad 27: Net-(BUS1-Pad27) -> unconnected-(BUS1-TC-Pad27)
- BUS1 pad 28: Net-(BUS1-Pad28) -> unconnected-(BUS1-ALE-Pad28)
- BUS1 pad 30: Net-(BUS1-Pad30) -> unconnected-(BUS1-OSC-Pad30)
- BUS1 pad 32: Net-(BUS1-Pad32) -> unconnected-(BUS1-IO_CH_CK-Pad32)
- BUS1 pad 5: Net-(BUS1-Pad5) -> unconnected-(BUS1--5V-Pad5)
- BUS1 pad 6: Net-(BUS1-Pad6) -> unconnected-(BUS1-DRQ2-Pad6)
- BUS1 pad 7: Net-(BUS1-Pad7) -> unconnected-(BUS1--12V-Pad7)
- BUS1 pad 8: Net-(BUS1-Pad8) -> unconnected-(BUS1-UNUSED-Pad8)
- BUS1 pad 9: Net-(BUS1-Pad9) -> unconnected-(BUS1-+12V-Pad9)
- J1 pad R7: Net-(J1-PadR7) -> unconnected-(J1-NC-PadR7)
- U1 pad 100: Net-(U1-Pad100) -> unconnected-(U1-INT4/IRQ10-Pad100)
- U1 pad 48: Net-(U1-Pad48) -> unconnected-(U1-TX--Pad48)
- U1 pad 49: Net-(U1-Pad49) -> unconnected-(U1-TX+-Pad49)
- U1 pad 53: Net-(U1-Pad53) -> unconnected-(U1-CD--Pad53)
- U1 pad 54: Net-(U1-Pad54) -> unconnected-(U1-CD+-Pad54)
- U1 pad 55: Net-(U1-Pad55) -> unconnected-(U1-RX--Pad55)
- U1 pad 56: Net-(U1-Pad56) -> unconnected-(U1-RX+-Pad56)
- U1 pad 60: Net-(U1-Pad60) -> unconnected-(U1-LEDBNC-Pad60)
- U1 pad 63: Net-(U1-Pad63) -> unconnected-(U1-LED2/LED_TX-Pad63)
- U1 pad 87: Net-(U1-Pad87) -> unconnected-(U1-SD15-Pad87)
- U1 pad 88: Net-(U1-Pad88) -> unconnected-(U1-SD14-Pad88)
- U1 pad 90: Net-(U1-Pad90) -> unconnected-(U1-SD13-Pad90)
- U1 pad 91: Net-(U1-Pad91) -> unconnected-(U1-SD12-Pad91)
- U1 pad 92: Net-(U1-Pad92) -> unconnected-(U1-SD11-Pad92)
- U1 pad 93: Net-(U1-Pad93) -> unconnected-(U1-SD10-Pad93)
- U1 pad 94: Net-(U1-Pad94) -> unconnected-(U1-SD9-Pad94)
- U1 pad 95: Net-(U1-Pad95) -> unconnected-(U1-SD8-Pad95)
- U1 pad 97: Net-(U1-Pad97) -> unconnected-(U1-INT7/IRQ15-Pad97)
- U1 pad 98: Net-(U1-Pad98) -> unconnected-(U1-INT6/IRQ12-Pad98)
- U1 pad 99: Net-(U1-Pad99) -> unconnected-(U1-INT5/IRQ11-Pad99)
- U3 pad 7: Net-(U3-Pad7) -> unconnected-(U3-NC-Pad7)
Routing:
- net GND: track 538.4 -> 0.00 mm, vias 26 -> 0
- net VCC: track 426.0 -> 0.00 mm, vias 16 -> 0
- net /~{SMEMW}: track 129.6 -> 0.00 mm, vias 1 -> 0
- net /~{SMEMR}: track 114.7 -> 0.00 mm, vias 1 -> 0
- net /A8: track 106.0 -> 0.00 mm, vias 1 -> 0
- net /A12: track 105.9 -> 0.00 mm, vias 1 -> 0
- net /A13: track 105.2 -> 0.00 mm, vias 1 -> 0
- net /A9: track 102.8 -> 0.00 mm, vias 1 -> 0
- net /A7: track 101.4 -> 0.00 mm, vias 1 -> 0
- net /A6: track 99.5 -> 0.00 mm, vias 1 -> 0
- net /A11: track 98.4 -> 0.00 mm, vias 1 -> 0
- net /A5: track 96.9 -> 0.00 mm, vias 1 -> 0
- net /A10: track 96.6 -> 0.00 mm, vias 1 -> 0
- net /A4: track 94.9 -> 0.00 mm, vias 1 -> 0
- net /A3: track 93.1 -> 0.00 mm, vias 1 -> 0
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- removed copper zone on B.Cu, net GND
- removed copper zone on F.Cu, net GND
- removed copper zone on B.Cu, net VCC
Other:
- net class Default removed
- net class Power removed
- board text removed: "5V"
- board text removed: "A0"
- board text removed: "A1"
- board text removed: "A10"
- board text removed: "A11"
- board text removed: "A12"
- board text removed: "A13"
- board text removed: "A14"
- board text removed: "A15"
- board text removed: "A16"
- board text removed: "A17"
- board text removed: "A19"
- board text removed: "A2"
- board text removed: "A20"
- board text removed: "A21"
- board text removed: "A3"
- board text removed: "A4"
- board text removed: "A5"
- board text removed: "A6"
- board text removed: "A7"
- board text removed: "A8"
- board text removed: "A9"
- board text removed: "D0"
- board text removed: "D1"
- board text removed: "D2"
- board text removed: "D3"
- board text removed: "D4"
- board text removed: "D5"
- board text removed: "D6"
- board text removed: "D7"
- board text removed: "GND"
- board text removed: "JLCJLCJLCJLC"
- board text removed: "NC"
- board text removed: "~CS"
- board text removed: "~MEMR"
- board text removed: "~MEMW"

Commit message: update 10102024
Parts:
- BUS1: footprint My_Components:Conn_Edge_PCB_ISA8 -> xt_eth:Conn_Edge_PCB_ISA8
- C1, C2, C3, C4, C5, C6, C7, C8: footprint Capacitor_THT:C_Disc_D7.0mm_W2.5mm_P5.00mm -> xt_eth:C_Disc_D7.0mm_W2.5mm_P5.00mm
- C10, C9: footprint Capacitor_THT:CP_Radial_D6.3mm_P2.50mm -> xt_eth:CP_Radial_D6.3mm_P2.50mm
- HOLE1, HOLE2: footprint MountingHole:MountingHole_3.2mm_M3_Pad_Via -> xt_eth:MountingHole_3.2mm_M3_Pad_Via
- J1: footprint Connector_RJ:RJ45_Amphenol_RJMG1BD3B8K1ANR -> xt_eth:RJ45_Amphenol_RJMG1BD3B8K1ANR
- J10: footprint Connector_PinHeader_2.54mm:PinHeader_2x05_P2.54mm_Vertical -> xt_eth:PinHeader_2x05_P2.54mm_Vertical
- J4, J7: footprint Connector_PinHeader_2.54mm:PinHeader_2x02_P2.54mm_Vertical -> xt_eth:PinHeader_2x02_P2.54mm_Vertical
- J9: footprint Connector_PinHeader_2.54mm:PinHeader_2x04_P2.54mm_Vertical -> xt_eth:PinHeader_2x04_P2.54mm_Vertical
- R1, R10, R11, R12, R13, R14, R15, R16, R17, R18, R19, R2, R3, R4, R5, R6, R7, R8, R9: footprint Resistor_THT:R_Axial_DIN0207_L6.3mm_D2.5mm_P10.16mm_Horizontal -> xt_eth:R_Axial_DIN0207_L6.3mm_D2.5mm_P10.16mm_Horizontal
- U1: footprint My_Components:IC_PQFP-100_14x20mm_P0.65mm_Hand_Soldering -> xt_eth:IC_PQFP-100_14x20mm_P0.65mm_Hand_Soldering
- U2: footprint My_Components:Socket_DIP32_600 -> xt_eth:Socket_DIP32_600
- U3: footprint Package_SO:SO-8_3.9x4.9mm_P1.27mm -> xt_eth:SO-8_3.9x4.9mm_P1.27mm
- Y1: footprint My_Components:Crystal_HC-49U_Vert -> xt_eth:Crystal_HC-49U_Vert
Routing:
- net GND: track 0.00 -> 451.9 mm
- net VCC: track 0.00 -> 337.0 mm, vias 0 -> 3
- net /~{SMEMW}: track 0.00 -> 133.0 mm, vias 0 -> 1
- net /BA16: track 0.00 -> 121.6 mm
- net /A12: track 0.00 -> 93.9 mm, vias 0 -> 1
- net /BA18: track 0.00 -> 93.3 mm
- net /A0: track 0.00 -> 93.2 mm
- net /A13: track 0.00 -> 89.1 mm, vias 0 -> 1
- net /A8: track 0.00 -> 87.9 mm, vias 0 -> 1
- net /A7: track 0.00 -> 87.6 mm, vias 0 -> 1
- net /~{SMEMR}: track 0.00 -> 86.4 mm, vias 0 -> 1
- net /A6: track 0.00 -> 85.1 mm, vias 0 -> 1
- net /A9: track 0.00 -> 84.4 mm, vias 0 -> 1
- net /A5: track 0.00 -> 83.1 mm, vias 0 -> 1
- net /BA17: track 0.00 -> 82.2 mm
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
Commit message: Version 0.1 ready gerbers
Routing:
- net /IRQ9: track 40.0 -> 40.6 mm
- net /~{IOR}: track 25.0 -> 25.6 mm
- net /~{IOW}: track 23.7 -> 24.2 mm
Other:
- board text added: "ISA 8-bit Ethernet Controller (TTH edition) (Original version by Sergey Kiselev (C), 2021) TTH edition ver 0.1 by MadCat https://github.com/madcatse/xt_ethernet https://t.me/madcatse https://www.youtube.com/@MadCatSE"
- board text added: "SW1"
- board text added: "SW2"
- board text added: "SW3"
- board text added: "SW4"
- board text removed: "Design files and documentation: github.com/skiselev/isa8_eth"
- board text removed: "Designed in Oregon"
- board text removed: "I/O Address 0x200 0x220 0x240 0x260 0x280 0x2A0 0x2C0 0x2E0"
- board text removed: "I/O Address 0x300 0x320 0x340 0x360 0x380 0x3A0 0x3C0 0x3E0"
- board text removed: "IRQ IRQ2 IRQ3 IRQ4 IRQ5"
- board text removed: "ISA 8-bit Ethernet Controller Version 1.0 Copyright (C) 2021 Sergey Kiselev"
- board text removed: "Licensed under CERN-OHL-S: https://cern-ohl.web.cern.ch"
- board text removed: "OFF: 16 KiB ROM ON: Page Mode"
- board text removed: "PnP"
- board text removed: "ROM Address Boot ROM Disabled 0xC0000 0xC4000 0xC8000 0xCC000 0xD0000 0xD4000 0xD8000 0xDC000 0xC0000 0xC8000 0xD0000 0xD8000 0xC0000 0xD0000"
- board text removed: "ROM Size 16 KiB 16 KiB 16 KiB 16 KiB 16 KiB 16 KiB 16 KiB 16 KiB 32 KiB 32 KiB 32 KiB 32 KiB 64 KiB 64 KiB"
- board text removed: "SW1.1: OFF - Jumperless; ON - Switches SW1.2: OFF - No PnP; ON - PnP Mode"
- board text removed: "SW2.1 OFF ON OFF ON"
- board text removed: "SW2.2 OFF OFF ON ON"
- board text removed: "SW3.1 OFF ON OFF ON OFF ON OFF ON"
- board text removed: "SW3.2 OFF OFF ON ON OFF OFF ON ON"
- board text removed: "SW3.3 OFF OFF OFF OFF OFF OFF OFF OFF"
- board text removed: "SW3.3 ON ON ON ON ON ON ON ON"
- board text removed: "SW3.4 OFF OFF OFF OFF ON ON ON ON"
- board text removed: "SW4.1 * OFF ON OFF ON OFF ON OFF ON OFF ON OFF ON OFF ON"
- board text removed: "SW4.2 * OFF OFF ON ON OFF OFF ON ON OFF OFF ON ON OFF OFF"
- board text removed: "SW4.3 * OFF OFF OFF OFF ON ON ON ON OFF OFF OFF OFF ON ON"
- board text removed: "SW4.4 OFF ON ON ON ON ON ON"
- board text removed: "SW4.5 OFF ON ON ON ON ON ON ON ON OFF OFF OFF OFF OFF OFF"
- board text removed: "Switches"
- board text removed: "www.malinov.com"
