File: KiCad/ISA8_Ethernet.kicad_pcb (KiCad board)
At the start: 2 copper layers, 104.1 x 74.9 mm, 41 parts, among them J1 RJMG1BD3B8K1ANR, J10 Conn_02x05_Odd_Even, J4 Conn_02x02_Odd_Even, J7 Conn_02x02_Odd_Even, J9 Conn_02x04_Odd_Even, U1 RTL8019AS, U2 SST39SF040, U3 93LC46C, Y1 20MHz

Commit message: Version 1.0 upload
Parts:
- C7: renamed from C3; value 0.01uF -> 10nF
- C8: renamed from C4; value 0.01uF -> 10nF
- J5: renamed from J1; value RJMG1BD3B8K1ANR -> HR911105A; footprint xt_eth:RJ45_Amphenol_RJMG1BD3B8K1ANR -> xt_eth:RJ45_HR911105A
- moved R10 21.1 mm to (154.5, 68.6), turned to -90 degrees
- moved C7 2.35 mm to (182.5, 92.7)
- moved C8 1.33 mm to (182.5, 96.5)
- moved Y1 0.30 mm to (180.2, 70.3)
- moved R18 0.17 mm to (200.4, 83.2)
- moved R11 0.10 mm to (158.6, 78.8)
- moved R12 0.10 mm to (161.7, 78.8)
- moved R13 0.10 mm to (164.8, 78.8)
- moved R14 0.10 mm to (167.9, 78.8)
- moved R15 0.10 mm to (171.0, 78.8)
- moved J3 0.06 mm to (142.0, 65.6)
- moved R6 0.06 mm to (141.1, 78.8)
- moved R7 0.06 mm to (144.2, 78.8)
- moved R8 0.06 mm to (147.3, 78.8)
- moved R9 0.06 mm to (150.4, 78.8)
- renumbered C10 to C1, C1 to C10, C7 to C2, C8 to C3, C6 to C4, C9 to C6, C2 to C9, J4 to J1, J7 to J2, J9 to J3, J10 to J4, R6 to R1, R18 to R10, R14 to R11, R15 to R12, R16 to R13, R17 to R14, R19 to R15, R7 to R16, R1 to R17, R3 to R18, R2 to R19, R4 to R2, R5 to R3, R8 to R4, R9 to R5, R10 to R6, R11 to R7, R12 to R8, R13 to R9, U2 to U1, U3 to U2, U1 to U3
Routing:
- net /AUI: track 5.46 -> 26.4 mm, vias 0 -> 1
- net GND: track 451.9 -> 460.6 mm
- net /A0: track 93.2 -> 84.7 mm, vias 0 -> 1
- net VCC: track 337.0 -> 342.7 mm
- net /BA18: track 93.3 -> 95.8 mm
- net Net-(J5-LEDG_K): track 8.23 -> 10.2 mm
- net /BD2: track 61.1 -> 62.6 mm
- net Net-(J5-LEDY_K): track 7.43 -> 8.86 mm
- net /TP_RX-: track 49.0 -> 50.4 mm
- net /~{SMEMW}: track 133.0 -> 134.4 mm
- net Net-(J5-RCT): track 16.7 -> 18.0 mm
- net /A15: track 25.9 -> 27.2 mm
- net /A16: track 24.1 -> 25.3 mm
- net /A8: track 87.9 -> 89.0 mm
- net /A9: track 84.4 -> 85.4 mm
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Other:
- board text added: "BOOT ROM"
- board text added: "Based on original version by Sergey Kiselev (C), 2021 https://github.com/skiselev/isa8_eth Thank you for an amazing card! ISA 8-bit Ethernet Controller (TTH edition) PCB board ver 1.0 by MadCat https://github.com/madcatse/xt_ethernet https://t.me/madcatse https://www.youtube.com/@MadCatSE"
- board text added: "EEPROM"
- board text added: "IF BOOT ROM NOT NEEDED, DO NOT PLACE: U1, SW4, R11-R15"
- board text added: "SW1 - CONFIG Jumperless: SW1.1 = 0, SW1.2 = 0 Jumpers: SW1.1 = 1, SW1.2 = 0 PnP: SW1.1 = 0, SW1.2 = 1"
- board text added: "SW2 - IRQ IRQ2/9 SW2.1 = 0, SW2.2 = 0 IRQ3 SW2.1 = 1, SW2.2 = 0 IRQ4 SW2.1 = 0, SW2.2 = 1 IRQ5 SW2.1 = 1, SW2.2 = 1"
- board text added: "SW3 - IO_ADDR I/O Add 3.1 3.2 3.3 3.4 0x200 0 0 1 0 0x220 1 0 1 0 0x240 0 1 1 0 0x260 1 1 1 0 0x280 0 0 1 1 0x2A0 1 0 1 1 0x2C0 0 1 1 1 0x2E0 1 1 1 1 0x300 0 0 0 0 0x320 1 0 0 0 0x340 0 1 0 0 0x360 1 1 0 0 0x380 0 0 0 1 0x3A0 1 0 0 1 0x3C0 0 1 0 1 0x3E0 1 1 0 1"
- board text removed: "ISA 8-bit Ethernet Controller (TTH edition) (Original version by Sergey Kiselev (C), 2021) TTH edition ver 0.1 by MadCat https://github.com/madcatse/xt_ethernet https://t.me/madcatse https://www.youtube.com/@MadCatSE"
