File: KiCad/ISA8_Ethernet.kicad_sch (KiCad schematic)
At the start: 41 parts, among them J1 RJMG1BD3B8K1ANR, J10 Conn_02x05_Odd_Even, J4 Conn_02x02_Odd_Even, J7 Conn_02x02_Odd_Even, J9 Conn_02x04_Odd_Even, U1 RTL8019AS, U2 SST39SF040, U3 93LC46C, Y1 20MHz

Commit message: Version 1.0 upload
Parts:
- BUS1: footprint My_Components:Conn_Edge_PCB_ISA8 -> xt_eth:Conn_Edge_PCB_ISA8
- C1: renamed from C10; footprint Capacitor_THT:CP_Radial_D6.3mm_P2.50mm -> xt_eth:CP_Radial_D6.3mm_P2.50mm
- C10: renamed from C1; footprint Capacitor_THT:C_Disc_D7.0mm_W2.5mm_P5.00mm -> xt_eth:C_Disc_D7.0mm_W2.5mm_P5.00mm
- C2: renamed from C7; footprint Capacitor_THT:C_Disc_D7.0mm_W2.5mm_P5.00mm -> xt_eth:C_Disc_D7.0mm_W2.5mm_P5.00mm
- C3: renamed from C8; footprint Capacitor_THT:C_Disc_D7.0mm_W2.5mm_P5.00mm -> xt_eth:C_Disc_D7.0mm_W2.5mm_P5.00mm
- C4: renamed from C6; footprint Capacitor_THT:C_Disc_D7.0mm_W2.5mm_P5.00mm -> xt_eth:C_Disc_D7.0mm_W2.5mm_P5.00mm
- C5: footprint Capacitor_THT:C_Disc_D7.0mm_W2.5mm_P5.00mm -> xt_eth:C_Disc_D7.0mm_W2.5mm_P5.00mm
- C6: renamed from C9; footprint Capacitor_THT:CP_Radial_D6.3mm_P2.50mm -> xt_eth:CP_Radial_D6.3mm_P2.50mm
- C7: renamed from C3; value 0.01uF -> 10nF; footprint Capacitor_THT:C_Disc_D7.0mm_W2.5mm_P5.00mm -> xt_eth:C_Disc_D7.0mm_W2.5mm_P5.00mm
- C8: renamed from C4; value 0.01uF -> 10nF; footprint Capacitor_THT:C_Disc_D7.0mm_W2.5mm_P5.00mm -> xt_eth:C_Disc_D7.0mm_W2.5mm_P5.00mm
- C9: renamed from C2; footprint Capacitor_THT:C_Disc_D7.0mm_W2.5mm_P5.00mm -> xt_eth:C_Disc_D7.0mm_W2.5mm_P5.00mm
- HOLE1, HOLE2: footprint MountingHole:MountingHole_3.2mm_M3_Pad_Via -> xt_eth:MountingHole_3.2mm_M3_Pad_Via
- J1: renamed from J4; footprint Connector_PinHeader_2.54mm:PinHeader_2x02_P2.54mm_Vertical -> xt_eth:PinHeader_2x02_P2.54mm_Vertical
- J2: renamed from J7; footprint Connector_PinHeader_2.54mm:PinHeader_2x02_P2.54mm_Vertical -> xt_eth:PinHeader_2x02_P2.54mm_Vertical
- J3: renamed from J9; footprint Connector_PinHeader_2.54mm:PinHeader_2x04_P2.54mm_Vertical -> xt_eth:PinHeader_2x04_P2.54mm_Vertical
- J4: renamed from J10; footprint Connector_PinHeader_2.54mm:PinHeader_2x05_P2.54mm_Vertical -> xt_eth:PinHeader_2x05_P2.54mm_Vertical
- J5: renamed from J1; value RJMG1BD3B8K1ANR -> HR911105A; footprint Connector_RJ:RJ45_Amphenol_RJMG1BD3B8K1ANR -> xt_eth:RJ45_HR911105A
- R1: renamed from R6; footprint Resistor_THT:R_Axial_DIN0207_L6.3mm_D2.5mm_P10.16mm_Horizontal -> xt_eth:R_Axial_DIN0207_L6.3mm_D2.5mm_P10.16mm_Horizontal
- R10: renamed from R18; footprint Resistor_THT:R_Axial_DIN0207_L6.3mm_D2.5mm_P10.16mm_Horizontal -> xt_eth:R_Axial_DIN0207_L6.3mm_D2.5mm_P10.16mm_Horizontal
- R11: renamed from R14; footprint Resistor_THT:R_Axial_DIN0207_L6.3mm_D2.5mm_P10.16mm_Horizontal -> xt_eth:R_Axial_DIN0207_L6.3mm_D2.5mm_P10.16mm_Horizontal
- R12: renamed from R15; footprint Resistor_THT:R_Axial_DIN0207_L6.3mm_D2.5mm_P10.16mm_Horizontal -> xt_eth:R_Axial_DIN0207_L6.3mm_D2.5mm_P10.16mm_Horizontal
- R13: renamed from R16; footprint Resistor_THT:R_Axial_DIN0207_L6.3mm_D2.5mm_P10.16mm_Horizontal -> xt_eth:R_Axial_DIN0207_L6.3mm_D2.5mm_P10.16mm_Horizontal
- R14: renamed from R17; footprint Resistor_THT:R_Axial_DIN0207_L6.3mm_D2.5mm_P10.16mm_Horizontal -> xt_eth:R_Axial_DIN0207_L6.3mm_D2.5mm_P10.16mm_Horizontal
- R15: renamed from R19; footprint Resistor_THT:R_Axial_DIN0207_L6.3mm_D2.5mm_P10.16mm_Horizontal -> xt_eth:R_Axial_DIN0207_L6.3mm_D2.5mm_P10.16mm_Horizontal
- R16: renamed from R7; footprint Resistor_THT:R_Axial_DIN0207_L6.3mm_D2.5mm_P10.16mm_Horizontal -> xt_eth:R_Axial_DIN0207_L6.3mm_D2.5mm_P10.16mm_Horizontal
- R17: renamed from R1; footprint Resistor_THT:R_Axial_DIN0207_L6.3mm_D2.5mm_P10.16mm_Horizontal -> xt_eth:R_Axial_DIN0207_L6.3mm_D2.5mm_P10.16mm_Horizontal
- R18: renamed from R3; footprint Resistor_THT:R_Axial_DIN0207_L6.3mm_D2.5mm_P10.16mm_Horizontal -> xt_eth:R_Axial_DIN0207_L6.3mm_D2.5mm_P10.16mm_Horizontal
- R19: renamed from R2; footprint Resistor_THT:R_Axial_DIN0207_L6.3mm_D2.5mm_P10.16mm_Horizontal -> xt_eth:R_Axial_DIN0207_L6.3mm_D2.5mm_P10.16mm_Horizontal
- R2: renamed from R4; footprint Resistor_THT:R_Axial_DIN0207_L6.3mm_D2.5mm_P10.16mm_Horizontal -> xt_eth:R_Axial_DIN0207_L6.3mm_D2.5mm_P10.16mm_Horizontal
- R3: renamed from R5; footprint Resistor_THT:R_Axial_DIN0207_L6.3mm_D2.5mm_P10.16mm_Horizontal -> xt_eth:R_Axial_DIN0207_L6.3mm_D2.5mm_P10.16mm_Horizontal
- R4: renamed from R8; footprint Resistor_THT:R_Axial_DIN0207_L6.3mm_D2.5mm_P10.16mm_Horizontal -> xt_eth:R_Axial_DIN0207_L6.3mm_D2.5mm_P10.16mm_Horizontal
- R5: renamed from R9; footprint Resistor_THT:R_Axial_DIN0207_L6.3mm_D2.5mm_P10.16mm_Horizontal -> xt_eth:R_Axial_DIN0207_L6.3mm_D2.5mm_P10.16mm_Horizontal
- R6: renamed from R10; footprint Resistor_THT:R_Axial_DIN0207_L6.3mm_D2.5mm_P10.16mm_Horizontal -> xt_eth:R_Axial_DIN0207_L6.3mm_D2.5mm_P10.16mm_Horizontal
- R7: renamed from R11; footprint Resistor_THT:R_Axial_DIN0207_L6.3mm_D2.5mm_P10.16mm_Horizontal -> xt_eth:R_Axial_DIN0207_L6.3mm_D2.5mm_P10.16mm_Horizontal
- R8: renamed from R12; footprint Resistor_THT:R_Axial_DIN0207_L6.3mm_D2.5mm_P10.16mm_Horizontal -> xt_eth:R_Axial_DIN0207_L6.3mm_D2.5mm_P10.16mm_Horizontal
- R9: renamed from R13; footprint Resistor_THT:R_Axial_DIN0207_L6.3mm_D2.5mm_P10.16mm_Horizontal -> xt_eth:R_Axial_DIN0207_L6.3mm_D2.5mm_P10.16mm_Horizontal
- U1: renamed from U2; footprint My_Components:Socket_DIP32_600 -> xt_eth:Socket_DIP32_600
- U2: renamed from U3; footprint Package_SO:SO-8_3.9x4.9mm_P1.27mm -> xt_eth:SO-8_3.9x4.9mm_P1.27mm
- U3: renamed from U1; footprint My_Components:IC_PQFP-100_14x20mm_P0.65mm_Hand_Soldering -> xt_eth:IC_PQFP-100_14x20mm_P0.65mm_Hand_Soldering
- Y1: footprint My_Components:Crystal_HC-49U_Vert -> xt_eth:Crystal_HC-49U_Vert
