File: KiCad/Version 2 (EthRTC)/ISA8_Ethernet.kicad_sch (KiCad schematic)
At the start: 52 parts, among them J1 Conn_02x02_Odd_Even, J2 Conn_02x02_Odd_Even, J3 Conn_02x04_Odd_Even, J4 Conn_02x05_Odd_Even, J5 HR911105A, J6 Conn_02x03_Odd_Even, U1 SST39SF040, U2 93LC46C, U3 RTL8019AS, U4 ATF16V8B, U5 DS12885, Y1 20MHz, Y2 32768Hz

Commit message: Update
Parts:
- removed RN1: 10k, Resistor_THT:R_Array_SIP5, symbol Eth_RTC:R_Network04
- added R20, R21, R22, R23: 10K, RTC_eth:R_Axial_DIN0207_L6.3mm_D2.5mm_P10.16mm_Horizontal, symbol Eth_RTC:R
- J6: footprint Connector_PinSocket_2.54mm:PinSocket_2x03_P2.54mm_Vertical -> Connector_PinHeader_2.54mm:PinHeader_2x03_P2.54mm_Vertical
Connections:
- net AS0: now also J6.6 (Pin_6), R20.1; no longer J6.2 (Pin_2)
- net AS1: now also R21.1
- net AS2: now also J6.2 (Pin_2), R22.1; no longer J6.6 (Pin_6)
- net VCC: now also J1.1 (Pin_1), J1.3 (Pin_3), J2.1 (Pin_1), J2.3 (Pin_3), J3.1 (Pin_1), J3.3 (Pin_3), J3.5 (Pin_5), J3.7 (Pin_7), J4.1 (Pin_1), J4.3 (Pin_3), J4.5 (Pin_5), J4.7 (Pin_7), J4.9 (Pin_9), R20.2, R21.2, R22.2, R23.2; no longer J1.2 (Pin_2), J1.4 (Pin_4), J2.2 (Pin_2), J2.4 (Pin_4), J3.2 (Pin_2), J3.4 (Pin_4), J3.6 (Pin_6), J3.8 (Pin_8), J4.10 (Pin_10), J4.2 (Pin_2), J4.4 (Pin_4), J4.6 (Pin_6), J4.8 (Pin_8)
- net ~{IRQ}: now also R23.1
- net at Y2.1: now also U5.3 (X2); no longer U5.2 (X1)
- net at Y2.2: now also U5.2 (X1); no longer U5.3 (X2)
- net at R8.2: now also J3.6 (Pin_6); no longer J3.5 (Pin_5)
- net at R9.2: now also J3.8 (Pin_8); no longer J3.7 (Pin_7)
- net at R11.2: now also J4.2 (Pin_2); no longer J4.1 (Pin_1)
- net at R4.2: now also J2.2 (Pin_2); no longer J2.1 (Pin_1)
- net at R5.2: now also J2.4 (Pin_4); no longer J2.3 (Pin_3)
- net at R15.2: now also J4.10 (Pin_10); no longer J4.9 (Pin_9)
- net at R13.2: now also J4.6 (Pin_6); no longer J4.5 (Pin_5)
- net at R12.2: now also J4.4 (Pin_4); no longer J4.3 (Pin_3)
- net at R6.2: now also J3.2 (Pin_2); no longer J3.1 (Pin_1)
- net at R7.2: now also J3.4 (Pin_4); no longer J3.3 (Pin_3)
- net at R2.2: now also J1.2 (Pin_2); no longer J1.1 (Pin_1)
- net at R3.2: now also J1.4 (Pin_4); no longer J1.3 (Pin_3)
- net at R14.2: now also J4.8 (Pin_8); no longer J4.7 (Pin_7)
