File: KiCad/Version 2 (EthRTC)/ISA8_Ethernet.kicad_pcb (KiCad board)
At the start: 2 copper layers, 136.7 x 76.9 mm, 55 parts, among them J1 Conn_02x02_Odd_Even, J2 Conn_02x02_Odd_Even, J3 Conn_02x04_Odd_Even, J4 Conn_02x05_Odd_Even, J5 HR911105A, J6 Conn_02x03_Odd_Even, U1 SST39SF040, U2 93LC46C, U3 RTL8019AS, U4 ATF16V8B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

Commit message: Silkscreen finish
Parts:
- added G***: LOGO, xt_eth:tme, B.Cu at (184.8, 71.6)
- added G1: LOGO, xt_eth:set_dont_get_it, B.Cu at (90.0, 118.2)
Routing:
- net /~{SMEMR}: track 121.1 -> 116.9 mm
Other:
- board text added: "1"
- board text added: "ATF16V8B"
- board text added: "Address 0x70 0x240 0x2A0 0x2C0 0x340 0x3A0 0x3C0"
- board text added: "Based on following projects github.com/skiselev/isa8_eth github.com/spark2k06/RTC8088 Thank you for an amazing cards! ISA 8-bit Ethernet Controller/RTC (TTH edition) PCB board ver 1.0 by MadCat https://github.com/madcatse/xt_ethernet https://t.me/madcatse https://www.youtube.com/@MadCatSE"
- board text added: "DS12885"
- board text added: "Ethermet Coonfig"
- board text added: "GAL POWER"
- board text added: "RTC Address Select"
- board text added: "RTC Power Switch"
- board text added: "SW4 - Consult https://github.com/skiselev/isa8_eth"
- board text added: "SW5"
- board text added: "SW5.1 OFF ON OFF ON OFF ON OFF"
- board text added: "SW5.2 OFF OFF ON ON OFF OFF ON"
- board text added: "SW5.3 OFF OFF OFF OFF ON ON ON"
- board text removed: "Based on original version by Sergey Kiselev (C), 2021 https://github.com/skiselev/isa8_eth Thank you for an amazing card! ISA 8-bit Ethernet Controller (TTH edition) PCB board ver 1.0 by MadCat https://github.com/madcatse/xt_ethernet https://t.me/madcatse https://www.youtube.com/@MadCatSE"

Commit message: Gerbers
Other:
- board text added: "Based on following projects github.com/skiselev/isa8_eth github.com/spark2k06/RTC8088 Thank you for amazing cards! ISA 8-bit Ethernet Controller/RTC (TTH edition) PCB board ver 1.0 by MadCat https://github.com/madcatse/xt_ethernet https://t.me/madcatse https://www.youtube.com/@MadCatSE"
- board text removed: "Based on following projects github.com/skiselev/isa8_eth github.com/spark2k06/RTC8088 Thank you for an amazing cards! ISA 8-bit Ethernet Controller/RTC (TTH edition) PCB board ver 1.0 by MadCat https://github.com/madcatse/xt_ethernet https://t.me/madcatse https://www.youtube.com/@MadCatSE"
Changed lines of the file:
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@@
 			(drillshape 0)
 			(scaleselection 1)
-			(outputdirectory "gerber")
+			(outputdirectory "gerber/")
 		)
 	)
@@
 		)
 	)
-	(gr_text "Based on following projects\ngithub.com/skiselev/isa8_eth\ngithub.com/spark2k06/RTC8088\nThank you for an amazing cards!\n\nISA 8-bit Ethernet Controller/RTC (TTH edition)\nPCB board ver 1.0 by MadCat\nhttps://github.com/madcatse/xt_ethernet\nhttps://t.me/madcatse\nhttps://www.youtube.com/@MadCatSE"
+	(gr_text "Based on following projects\ngithub.com/skiselev/isa8_eth\ngithub.com/spark2k06/RTC8088\nThank you for amazing cards!\n\nISA 8-bit Ethernet Controller/RTC (TTH edition)\nPCB board ver 1.0 by MadCat\nhttps://github.com/madcatse/xt_ethernet\nhttps://t.me/madcatse\nhttps://www.youtube.com/@MadCatSE"
 		(at 128.4732 107.5944 0)
 		(layer "B.SilkS")
